Commit message: reworking configs

File: src/puma560_description/urdf/puma560_robot.urdf.xacro (robot description, xacro)
@@ -1,7 +1,6 @@
 <?xml version="1.0"?>
 <robot name="Puma560" xmlns:xacro="http://www.ros.org/wiki/xacro">
-    <xacro:property name="mesh_dir" value="package://puma560_description/meshes"/>
-    <xacro:macro name="puma560_link_geometry" params="link_num">
-        <mesh filename="${mesh_dir}/puma_link${link_num}.stl" scale="${0.1*25.4} ${0.1*25.4} ${0.1*25.4}"/>
+    <xacro:macro name="robot_mesh" params="name">
+        <mesh filename="package://puma560_description/meshes/${name}" scale="${0.001*25.4} ${0.001*25.4} ${0.001*25.4}"/>
     </xacro:macro>
     <material name="blue">
@@ -14,126 +13,196 @@
         <color rgba="0 0.8 0 0.8"/>
     </material>
-    <xacro:property name="M_PI" value="3.14159265"/>
-    <xacro:property name="d_1" value="0.6718"/>
-    <xacro:property name="d_2" value="0.1501"/>
-    <xacro:property name="d_3" value="0"/>
-    <xacro:property name="d_4" value="0.4331"/>
-    <xacro:property name="d_5" value="0"/>
-    <xacro:property name="d_6" value="0.0558"/>
-    <xacro:property name="a_1" value="0"/>
-    <xacro:property name="a_2" value="0.4318"/>
-    <xacro:property name="a_3" value="-0.0203"/>
-    <xacro:property name="a_4" value="0"/>
-    <xacro:property name="a_5" value="0"/>
-    <xacro:property name="a_6" value="0"/>
-    <xacro:macro name="link" params="num color vxyz vrpy cxyz crpy ixyz irpy mass ixx ixy ixz iyy iyz izz">
-      <link name="link${num}">
-        <visual>
-          <geometry>
-            <xacro:puma560_link_geometry link_num="${num}"/>
-          </geometry>
-          <origin xyz="${vxyz}" rpy="${vrpy}"/>
-          <material name="${color}"/>
-        </visual>
-        <collision>
-          <geometry>
-            <xacro:puma560_link_geometry link_num="${num}"/>
-          </geometry>
-          <origin xyz="${cxyz}" rpy="${crpy}"/>
-        </collision>
-        <inertial>
-            <origin xyz="${ixyz}" rpy="${irpy}"/>
-            <mass value="${mass}"/>
-            <inertia ixx="${ixx}" ixy="${ixy}" ixz="${ixz}" iyy="${iyy}" iyz="${iyz}" izz="${izz}"/>
-        </inertial>
-      </link>
-    </xacro:macro>
-    <xacro:macro name="joint" params="name type parent child xyz rpy axyz effort lower upper velocity damping friction">
-        <joint name="${name}" type="${type}">
-            <parent link="${parent}"/>
-            <child link="${child}"/>
-            <origin xyz="${xyz}" rpy="${rpy}"/>
-            <axis xyz="${axyz}"/>
-            <limit effort="${effort}" lower="${lower}" upper="${upper}" velocity="${velocity}"/>
-            <dynamics damping="${damping}" friction="${friction}"/>
-        </joint>
-    </xacro:macro>
     <link name="world"/>
-    <xacro:link num="1" color="green"
-                vxyz="0 0 0" vrpy="0 0 ${M_PI/2}"
-                cxyz="0 0 0" crpy="0 0 ${M_PI/2}"
-                ixyz="0 0 0" irpy="0 0 0"
-                mass="1.0"
-                ixx="0.001" ixy="0" ixz="0" iyy="0.001" iyz="0" izz="0.001"/>
-    <xacro:link num="2" color="red"
-                vxyz="0 0 -0.1" vrpy="0 0 0"
-                cxyz="0 0 0" crpy="0 0 ${M_PI/2}"
-                ixyz="0 0 0" irpy="0 0 0"
-                mass="1.0"
-                ixx="0.001" ixy="0" ixz="0" iyy="0.001" iyz="0" izz="0.001"/>
-    <xacro:link num="3" color="blue"
-                vxyz="0 0 ${0.0435+d_2}" vrpy="0 0 0"
-                cxyz="0 0 0" crpy="0 0 ${M_PI/2}"
-                ixyz="0 0 0" irpy="0 0 0"
-                mass="1.0"
-                ixx="0.001" ixy="0" ixz="0" iyy="0.001" iyz="0" izz="0.001"/>
-    <xacro:link num="4" color="green"
-                vxyz="0 0 0" vrpy="0 0 0"
-                cxyz="0 0 0" crpy="0 0 ${M_PI/2}"
-                ixyz="0 0 0" irpy="0 0 0"
-                mass="1.0"
-                ixx="0.001" ixy="0" ixz="0" iyy="0.001" iyz="0" izz="0.001"/>
-    <xacro:link num="5" color="red"
-                vxyz="0 0 ${d_4-0.071}" vrpy="0 0 ${M_PI/2}"
-                cxyz="0 0 0" crpy="0 0 ${M_PI/2}"
-                ixyz="0 0 0" irpy="0 0 0"
-                mass="1.0"
-                ixx="0.001" ixy="0" ixz="0" iyy="0.001" iyz="0" izz="0.001"/>
-    <xacro:link num="6" color="green"
-                vxyz="0 0 0" vrpy="${M_PI} 0 ${M_PI/2}"
-                cxyz="0 0 0" crpy="0 0 ${M_PI/2}"
-                ixyz="0 0 0" irpy="0 0 0"
-                mass="1.0"
-                ixx="0.001" ixy="0" ixz="0" iyy="0.001" iyz="0" izz="0.001"/>
-    <xacro:link num="7" color="blue"
-                vxyz="0 0 -0.010" vrpy="0 0 0"
-                cxyz="0 0 0" crpy="0 0 ${M_PI/2}"
-                ixyz="0 0 0" irpy="0 0 0"
-                mass="1.0"
-                ixx="0.001" ixy="0" ixz="0" iyy="0.001" iyz="0" izz="0.001"/>
-    <xacro:joint name="world_to_link1" type="fixed" parent="world" child="link1"
-                 xyz="0 0 0" rpy="0 0 0"
-                 axyz="0 0 0"
-                 effort="0" lower="0" upper="0" velocity="0"
-                 damping="0" friction="0"/>
-    <xacro:joint name="j1" type="revolute" parent="link1" child="link2"
-                 xyz="0 0 ${d_1}" rpy="${M_PI/2} 0 0"
-                 axyz="0 1 0"
-                 effort="1000.0" lower="${-M_PI}" upper="${M_PI}" velocity="2.0"
-                 damping="1.0" friction="0.1"/>
-    <xacro:joint name="j2" type="revolute" parent="link2" child="link3"
-                 xyz="0 0 0" rpy="0 0 0"
-                 axyz="0 0 1"
-                 effort="1000.0" lower="${-M_PI/2}" upper="${M_PI/2}" velocity="2.0"
-                 damping="1.0" friction="0.1"/>
-    <xacro:joint name="j3" type="revolute" parent="link3" child="link4"
-                 xyz="${a_2} ${a_3} ${d_2}" rpy="0 0 ${-M_PI/2}"
-                 axyz="0 0 1"
-                 effort="1000.0" lower="${-M_PI/2}" upper="${M_PI/2}" velocity="2.0"
-                 damping="1.0" friction="0.1"/>
-    <xacro:joint name="j4" type="revolute" parent="link4" child="link5"
-                 xyz="0 0 0" rpy="${M_PI/2} 0 ${M_PI/2}"
-                 axyz="0 0 1"
-                 effort="1000.0" lower="${-M_PI/2}" upper="${M_PI/2}" velocity="2.0"
-                 damping="1.0" friction="0.1"/>
-    <xacro:joint name="j5" type="revolute" parent="link5" child="link6"
-                 xyz="0 0 ${d_4}" rpy="${M_PI/2} 0 0"
-                 axyz="0 0 1"
-                 effort="1000.0" lower="${-M_PI/2}" upper="${M_PI/2}" velocity="2.0"
-                 damping="1.0" friction="0.1"/>
-    <xacro:joint name="j6" type="revolute" parent="link6" child="link7"
-                 xyz="0 ${d_6} 0" rpy="${-M_PI/2} 0 0"
-                 axyz="0 0 1"
-                 effort="1000.0" lower="${-M_PI/2}" upper="${M_PI/2}" velocity="2.0"
-                 damping="1.0" friction="0.1"/>
+    <link name="link1">
+        <visual>
+            <geometry>
+                <xacro:robot_mesh name="puma_link1.stl"/>
+            </geometry>
+            <origin rpy="0 0 1.570796325"/>
+            <material name="green"/>
+        </visual>
+        <collision>
+            <geometry>
+                <xacro:robot_mesh name="puma_link1.stl"/>
+            </geometry>
+            <origin rpy="0 0 1.570796325"/>
+        </collision>
+        <inertial>
+            <origin xyz="0 0 0" rpy="0 0 0"/>
+            <mass value="100.0"/>
+            <inertia ixx="1.0" ixy="0.0" ixz="0.0" iyy="1.0" iyz="0.0" izz="1.0"/>
+        </inertial>
+    </link>
+    <link name="link2">
+        <visual>
+            <geometry>
+                <xacro:robot_mesh name="puma_link2.stl"/>
+            </geometry>
+            <origin xyz="0 0 -0.1"/>
+            <material name="red"/>
+        </visual>
+        <collision>
+            <geometry>
+                <xacro:robot_mesh name="puma_link2.stl"/>
+            </geometry>
+            <origin xyz="0 0 -0.1"/>
+        </collision>
+        <inertial>
+            <origin xyz="0 0 0" rpy="0 0 0"/>
+            <mass value="0.1"/>
+            <inertia ixx="1.0" ixy="0.0" ixz="0.0" iyy="1.0" iyz="0.0" izz="1.0"/>
+        </inertial>
+    </link>
+    <link name="link3">
+        <visual>
+            <geometry>
+                <xacro:robot_mesh name="puma_link3.stl"/>
+            </geometry>
+            <origin xyz="0 0 0.1936"/>
+            <material name="blue"/>
+        </visual>
+        <collision>
+            <geometry>
+                <xacro:robot_mesh name="puma_link3.stl"/>
+            </geometry>
+            <origin xyz="0 0 0.1936"/>
+        </collision>
+        <inertial>
+            <origin xyz="0 0 0" rpy="0 0 0"/>
+            <mass value="0.1"/>
+            <inertia ixx="1.0" ixy="0.0" ixz="0.0" iyy="1.0" iyz="0.0" izz="1.0"/>
+        </inertial>
+    </link>
+    <link name="link4">
+        <visual>
+            <geometry>
+                <xacro:robot_mesh name="puma_link4.stl"/>
+            </geometry>
+            <origin xyz="0 0 0"/>
+            <material name="green"/>
+        </visual>
+        <collision>
+            <geometry>
+                <xacro:robot_mesh name="puma_link4.stl"/>
+            </geometry>
+            <origin xyz="0 0 0"/>
+        </collision>
+        <inertial>
+            <origin xyz="0 0 0" rpy="0 0 0"/>
+            <mass value="0.1"/>
+            <inertia ixx="1.0" ixy="0.0" ixz="0.0" iyy="1.0" iyz="0.0" izz="1.0"/>
+        </inertial>
+    </link>
+    <link name="link5">
+        <visual>
+            <geometry>
+                <xacro:robot_mesh name="puma_link5.stl"/>
+            </geometry>
+            <origin rpy="0 0 1.570796325" xyz="0 0 0.3621"/>
+            <material name="red"/>
+        </visual>
+        <collision>
+            <geometry>
+                <xacro:robot_mesh name="puma_link5.stl"/>
+            </geometry>
+            <origin rpy="0 0 1.570796325" xyz="0 0 0.3621"/>
+        </collision>
+        <inertial>
+            <origin xyz="0 0 0" rpy="0 0 0"/>
+            <mass value="0.1"/>
+            <inertia ixx="1.0" ixy="0.0" ixz="0.0" iyy="1.0" iyz="0.0" izz="1.0"/>
+        </inertial>
+    </link>
+    <link name="link6">
+        <visual>
+            <geometry>
+                <xacro:robot_mesh name="puma_link6.stl"/>
+            </geometry>
+            <origin rpy="3.14159265 0 1.570796325"/>
+            <material name="green"/>
+        </visual>
+        <collision>
+            <geometry>
+                <xacro:robot_mesh name="puma_link6.stl"/>
+            </geometry>
+            <origin rpy="3.14159265 0 1.570796325"/>
+        </collision>
+        <inertial>
+            <origin xyz="0 0 0" rpy="0 0 0"/>
+            <mass value="0.1"/>
+            <inertia ixx="1.0" ixy="0.0" ixz="0.0" iyy="1.0" iyz="0.0" izz="1.0"/>
+        </inertial>
+    </link>
+    <link name="link7">
+        <visual>
+            <geometry>
+                <xacro:robot_mesh name="puma_link7.stl"/>
+            </geometry>
+            <origin xyz="0 0 -0.010"/>
+            <material name="blue"/>
+        </visual>
+        <collision>
+            <geometry>
+                <xacro:robot_mesh name="puma_link7.stl"/>
+            </geometry>
+            <origin xyz="0 0 -0.010"/>
+        </collision>
+        <inertial>
+            <origin xyz="0 0 0" rpy="0 0 0"/>
+            <mass value="0.1"/>
+            <inertia ixx="1.0" ixy="0.0" ixz="0.0" iyy="1.0" iyz="0.0" izz="1.0"/>
+        </inertial>
+    </link>
+    <joint name="base" type="fixed">
+        <parent link="world"/>
+        <child link="link1"/>
+    </joint>
+    <joint name="join1" type="revolute">
+        <parent link="link1"/>
+        <child link="link2"/>
+        <origin xyz="0 0 0.6718" rpy="1.570796325 0 0"/>
+        <axis xyz="0 1 0"/>
+        <limit effort="1000.0" lower="-3.14159265" upper="3.14159265" velocity="2.0"/>
+        <dynamics damping="1.0" friction="0.1"/>
+    </joint>
+    <joint name="join2" type="revolute">
+        <parent link="link2"/>
+        <child link="link3"/>
+        <origin xyz="0 0 0" rpy="0 0 0"/>
+        <axis xyz="0 0 1"/>
+        <limit effort="1000.0" lower="-1.570796325" upper="1.570796325" velocity="2.0"/>
+        <dynamics damping="1.0" friction="0.1"/>
+    </joint>
+    <joint name="join3" type="revolute">
+        <parent link="link3"/>
+        <child link="link4"/>
+        <origin xyz="0.4318 -0.0203 0.1501" rpy="0 0 -1.570796325"/>
+        <axis xyz="0 0 1"/>
+        <limit effort="1000.0" lower="-1.570796325" upper="1.570796325" velocity="2.0"/>
+        <dynamics damping="1.0" friction="0.1"/>
+    </joint>
+    <joint name="join4" type="revolute">
+        <parent link="link4"/>
+        <child link="link5"/>
+        <origin xyz="0 0 0" rpy="1.570796325 0 1.570796325"/>
+        <axis xyz="0 0 1"/>
+        <limit effort="1000.0" lower="-1.570796325" upper="1.570796325" velocity="2.0"/>
+        <dynamics damping="1.0" friction="0.1"/>
+    </joint>
+    <joint name="join5" type="revolute">
+        <parent link="link5"/>
+        <child link="link6"/>
+        <origin xyz="0 0 0.4331" rpy="1.570796325 0 0"/>
+        <axis xyz="0 0 1"/>
+        <limit effort="1000.0" lower="-1.570796325" upper="1.570796325" velocity="2.0"/>
+        <dynamics damping="1.0" friction="0.1"/>
+    </joint>
+    <joint name="join6" type="revolute">
+        <parent link="link6"/>
+        <child link="link7"/>
+        <origin xyz="0 0.0558 0" rpy="-1.570796325 0 0"/>
+        <axis xyz="0 0 1"/>
+        <limit effort="1000.0" lower="-1.570796325" upper="1.570796325" velocity="2.0"/>
+        <dynamics damping="1.0" friction="0.1"/>
+    </joint>
 </robot>
